File: circuit/OSASU_Keyboard.kicad_sch (KiCad schematic)
At the start: 5 parts, among them J1 Conn_01x05_Pin, J2 Conn_01x05_Socket, J3 Conn_01x05_Pin, J4 Conn_01x05_Socket, J5 Conn_01x05_Pin

Commit message: PCB更新
Parts:
- J2, J4: footprint Connector_PinHeader_1.27mm:PinHeader_1x05_P1.27mm_Horizontal -> Connector_PinSocket_1.27mm:PinSocket_1x05_P1.27mm_Vertical
- J3, J5: footprint custom:PinHeader_1x05_P2.54mm_Right_angle -> Connector_PinHeader_1.27mm:PinHeader_1x05_P1.27mm_Horizontal
Changed lines of the file:
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@@
 			)
 		)
-		(property "Footprint" "Connector_PinHeader_1.27mm:PinHeader_1x05_P1.27mm_Horizontal"
+		(property "Footprint" "Connector_PinSocket_1.27mm:PinSocket_1x05_P1.27mm_Vertical"
 			(at 181.61 91.44 0)
 			(hide yes)
@@
 			)
 		)
-		(property "Footprint" "custom:PinHeader_1x05_P2.54mm_Right_angle"
+		(property "Footprint" "Connector_PinHeader_1.27mm:PinHeader_1x05_P1.27mm_Horizontal"
 			(at 193.04 102.87 0)
 			(hide yes)
@@
 			)
 		)
-		(property "Footprint" "Connector_PinHeader_1.27mm:PinHeader_1x05_P1.27mm_Horizontal"
+		(property "Footprint" "Connector_PinSocket_1.27mm:PinSocket_1x05_P1.27mm_Vertical"
 			(at 110.49 91.44 0)
 			(hide yes)
@@
 			)
 		)
-		(property "Footprint" "custom:PinHeader_1x05_P2.54mm_Right_angle"
+		(property "Footprint" "Connector_PinHeader_1.27mm:PinHeader_1x05_P1.27mm_Horizontal"
 			(at 157.48 91.44 0)
 			(hide yes)
