File: circuit/OSASU_Keyboard.kicad_pcb (KiCad board)
At the start: 2 copper layers, 19.1 x 19 mm, 17 parts, among them J1 Conn_01x05_Pin, J2 Conn_01x05_Socket, J3 Conn_01x05_Pin, P1 USB_C_Plug_USB2.0, SW1 SW_Push, SW2 SW_Push, U1 CH552T, U2 CH32V003FxPx

Commit message: commit
Parts:
- removed SW1: SW_Push, Button_Switch_Keyboard:SW_Cherry_MX_1.00u_PCB
- C3, J2, J3, U2: moved to B.Cu
- moved D1 71.5 mm to (201.8, 79.7)
- moved SW2 63.4 mm to (205.1, 87.9)
- moved U2 51.1 mm to (202.6, 98.7), turned to 180 degrees
- moved C3 47.4 mm to (195.4, 84.7), turned to 180 degrees
- moved C1 32.8 mm to (177.6, 86.3), turned to -90 degrees
- moved R3 26.8 mm to (173.5, 93.7)
- moved P1 23.4 mm to (144.1, 102.3)
- moved C2 21.2 mm to (147.9, 94.0), turned to 90 degrees
- moved U1 20.6 mm to (171.6, 88.4)
- moved R1 17.6 mm to (141.9, 94.0), turned to 90 degrees
- moved R2 14.7 mm to (143.4, 94.0), turned to 90 degrees
- moved R4 8.98 mm to (146.4, 94.0), turned to 90 degrees
- moved R5 7.33 mm to (144.9, 94.0), turned to 90 degrees
- moved J3 5.53 mm to (210.5, 96.1)
- moved J1 4.53 mm to (179.5, 90.3)
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Other:
- board size 19.1 x 19 mm -> 49.5 x 19.1 mm

Commit message: commit
Parts:
- added JP1: Jumper_2_Open, Jumper:SolderJumper-2_P1.3mm_Open_RoundedPad1.0x1.5mm, B.Cu at (179.3, 101.0)
- C2, J1, P1, R1, R2, R3, R4, R5, U1: moved to B.Cu
- D1: footprint LED_THT:LED_D5.0mm -> LED_SMD:LED_Yuji_5730
- moved P1 31.9 mm to (172.2, 87.1)
- moved R1 23.8 mm to (165.6, 95.3), turned to 0 degrees
- moved C2 23.5 mm to (171.4, 93.5), turned to 180 degrees
- moved R2 22.2 mm to (165.6, 93.8), turned to 0 degrees
- moved R5 20.9 mm to (165.0, 99.7)
- moved D1 19.1 mm to (202.8, 98.8)
- moved R4 18.0 mm to (163.5, 99.7)
- moved C3 11.7 mm to (196.8, 96.3), turned to 90 degrees
- moved U1 9.98 mm to (171.3, 98.4)
- moved C1 7.81 mm to (176.3, 94.0), turned to 90 degrees
- moved R3 7.56 mm to (176.8, 100.5), turned to 90 degrees
- moved J1 5.24 mm to (180.1, 95.5)
- moved J2 0.75 mm to (194.7, 90.4)
- moved J3 0.59 mm to (210.5, 95.5)
- moved U2 0.15 mm to (202.7, 98.8)

Commit message: commit
Parts:
- J3: footprint Connector_PinHeader_1.27mm:PinHeader_1x05_P1.27mm_Horizontal -> custom:PinHeader_1x05_P2.54mm_Right_angle
- moved J3 4.19 mm to (208.0, 98.9)

Commit message: schematicを更新
Parts:
- added J4: Conn_01x05_Socket, Connector_PinHeader_1.27mm:PinHeader_1x05_P1.27mm_Horizontal, F.Cu at (253.3, 102.9)
- added J5: Conn_01x05_Pin, custom:PinHeader_1x05_P2.54mm_Right_angle, F.Cu at (250.9, 88.8)
- C2, C3, J1, J2, J3, JP1, P1, R1, R2, R3, R4, R5, U1, U2: moved to F.Cu
- moved P1 79.1 mm to (245.4, 116.9)
- moved C3 78.4 mm to (266.4, 132.6), turned to 0 degrees
- moved R4 78.3 mm to (237.4, 125.5), turned to 0 degrees
- moved U1 78.0 mm to (244.3, 125.7)
- moved R5 77.7 mm to (237.4, 128.0), turned to 0 degrees
- moved R2 76.6 mm to (237.4, 120.4)
- moved R1 75.3 mm to (237.4, 117.9)
- moved JP1 75.0 mm to (250.9, 123.4), turned to 0 degrees
- moved D1 72.2 mm to (268.4, 129.0)
- moved C2 69.5 mm to (237.4, 115.4), turned to 0 degrees
- moved SW2 65.5 mm to (265.2, 114.1)
- moved U2 65.4 mm to (259.8, 130.8), turned to 0 degrees
- moved R3 64.6 mm to (237.4, 123.0), turned to 0 degrees
- moved C1 64.0 mm to (237.4, 112.9), turned to 0 degrees
- moved J1 57.3 mm to (236.9, 102.9)
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Connections:
- net /Adress_{(Sink)}⇒ renamed /Sleve/Adress(Sink)
- net /Adress_{(Source)} ⇒ Adress_{(Sink)} renamed /HOST/Adress_{(Source)} ⇒ Adress_{(Sink)}
- net /D+_{(USB)} = UDP_{(CH552)} renamed /HOST/D+_{(USB)} = UDP_{(CH552)}
- net /D-_{(USB)} = UDM_{(CH552)} renamed /HOST/D-_{(USB)} = UDM_{(CH552)}
- net /LED⇒  renamed /Sleve/LED⇒ 
- net /SW1 renamed /Sleve/SW1
- net /⇒Adress_{(Slave)} renamed /Sleve/Adress(Slave)
- J1 pad 2: /SCL_{(CH552T)} = SCL_{(CH32V003)} -> /HOST/SDA_{(CH552T)} = SDA_{(CH32V003)}
- J1 pad 3: /SDA_{(CH552T)} = SDA_{(CH32V003)} -> /HOST/SCL_{(CH552T)} = SCL_{(CH32V003)}
- J2 pad 2: /⇒ PC1 -> /Sleve/PC2
- J2 pad 3: /⇒ PC2 -> /Sleve/PC1
- J3 pad 2: /⇒ PC1 -> /Sleve/PC2
- J3 pad 3: /⇒ PC2 -> /Sleve/PC1
- R4 pad 2: /SCL_{(CH552T)} = SCL_{(CH32V003)} -> /HOST/SCL_{(CH552T)} = SCL_{(CH32V003)}
- R5 pad 2: /SDA_{(CH552T)} = SDA_{(CH32V003)} -> /HOST/SDA_{(CH552T)} = SDA_{(CH32V003)}
- U1 pad 4: /SDA_{(CH552T)} = SDA_{(CH32V003)} -> /HOST/SDA_{(CH552T)} = SDA_{(CH32V003)}
- U1 pad 5: /SCL_{(CH552T)} = SCL_{(CH32V003)} -> /HOST/SCL_{(CH552T)} = SCL_{(CH32V003)}
- U2 pad 11: /⇒ PC1 -> /Sleve/PC1
- U2 pad 12: /⇒ PC2 -> /Sleve/PC2

Commit message: PCB更新
Parts:
- J2, J4: footprint Connector_PinHeader_1.27mm:PinHeader_1x05_P1.27mm_Horizontal -> Connector_PinSocket_1.27mm:PinSocket_1x05_P1.27mm_Vertical
- J3, J5: footprint custom:PinHeader_1x05_P2.54mm_Right_angle -> Connector_PinHeader_1.27mm:PinHeader_1x05_P1.27mm_Horizontal
- moved SW2 94.2 mm to (174.7, 87.8)
- moved J2 46.5 mm to (199.1, 96.3)
- moved J1 27.8 mm to (209.9, 96.3)
- moved J4 21.3 mm to (274.3, 99.4)
- moved J5 21.3 mm to (271.9, 85.2)
Other:
- board size 49.5 x 19.1 mm -> 49.2 x 19.2 mm

Commit message: 基盤更新
Parts:
- moved U1 96.9 mm to (147.6, 130.0)
- moved P1 95.9 mm to (149.6, 119.7), turned to 180 degrees
- moved R4 95.8 mm to (141.7, 129.0), turned to -90 degrees
- moved R2 93.5 mm to (144.0, 125.5), turned to 180 degrees
- moved R1 89.9 mm to (147.8, 125.5)
- moved C1 84.9 mm to (153.5, 125.7)
- moved C2 84.9 mm to (153.4, 127.5)
- moved R5 84.4 mm to (153.2, 131.8), turned to -90 degrees
- moved R3 80.2 mm to (157.4, 118.4)
- moved J1 59.4 mm to (156.8, 122.9)
- moved J5 26.6 mm to (245.7, 90.2), turned to -90 degrees
- turned J3 to 180 degrees
Other:
- board size 49.2 x 19.2 mm -> 71.6 x 51.7 mm
