File: PCB/OSASU_Keyboard.kicad_sch (KiCad schematic)
At the start: 5 parts, among them J1 Conn_01x05_Pin, J2 Conn_01x05_Socket, J3 Conn_01x05_Pin, J4 Conn_01x05_Socket, J5 Conn_01x05_Pin

Commit message: 基盤設計
Parts:
- removed J4: Conn_01x05_Socket, Connector_PinSocket_1.27mm:PinSocket_1x05_P1.27mm_Vertical, symbol Connector:Conn_01x05_Socket
- removed J5: Conn_01x05_Pin, Connector_PinHeader_1.27mm:PinHeader_1x05_P1.27mm_Horizontal, symbol Connector:Conn_01x05_Pin
- J1, J3: footprint Connector_PinHeader_1.27mm:PinHeader_1x05_P1.27mm_Horizontal -> custom:PinHeader_1x05_P1.27mm_Horizontal_SMD(inversed)
- J2: footprint Connector_PinSocket_1.27mm:PinSocket_1x05_P1.27mm_Vertical -> custom:PinHeader_1x05_P1.27mm_Horizontal_SMD
Other:
- title: (none) -> OSASU-keyboard
