File: PCB/OSASU_Keyboard.kicad_sch (KiCad schematic)
At the start: 4 parts, among them J1 Conn_01x05_Pin, J2 Conn_01x05_Socket, J3 Conn_01x05_Pin

Commit message: commit
Changed lines of the file:
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@@
 	(symbol
 		(lib_id "Graphic:SYM_EasterEgg_42x60mm")
-		(at 80.01 179.07 0)
+		(at 74.93 76.2 0)
 		(unit 1)
 		(body_style 1)
@@
 		(fields_autoplaced yes)
 		(property "Reference" "SYM1"
-			(at 80.01 179.07 0)
+			(at 74.93 76.2 0)
 			(hide yes)
 			(show_name no)
@@
 		)
 		(property "Value" "SYM_EasterEgg_42x60mm"
-			(at 80.01 179.07 0)
+			(at 74.93 76.2 0)
 			(hide yes)
 			(show_name no)
@@
 		)
 		(property "Footprint" "Symbol:EasterEgg_EWG1308-2013_ClassA"
-			(at 80.01 182.88 0)
+			(at 74.93 80.01 0)
 			(hide yes)
 			(show_name no)
@@
 		)
 		(property "Datasheet" "https://eur-lex.europa.eu/LexUriServ/LexUriServ.do?uri=OJ:L:2013:347:0671:0854:de:PDF"
-			(at 80.01 185.42 0)
+			(at 74.93 82.55 0)
 			(hide yes)
 			(show_name no)
@@
 		)
 		(property "Description" "EasterEgg, ClassA, Medium Size"
-			(at 80.01 179.07 0)
+			(at 74.93 76.2 0)
 			(hide yes)
 			(show_name no)
