File: PCB/host.kicad_sch (KiCad schematic)
At the start: 10 parts, among them P1 USB_C_Plug_USB2.0, U1 CH552T

Commit message: 基盤設計
Parts:
- added F1: Fuse 350mA 15V, Fuse:Fuse_0603_1608Metric, symbol Device:Fuse_Small
- added J5: Conn_01x03, Connector_PinHeader_2.54mm:PinHeader_1x03_P2.54mm_Vertical, symbol Connector_Generic:Conn_01x03
- added JP2: Jumper_2_Open, Jumper:SolderJumper-2_P1.3mm_Open_RoundedPad1.0x1.5mm, symbol Jumper:Jumper_2_Open
- R3: value 10k -> 2.2k
Connections:
- net +3V3: now also J5.2 (Pin_2)
- net +5V: now also F1.2, J5.1 (Pin_1), JP2.2 (B); no longer P1.A4 (VBUS), P1.A9 (VBUS), P1.B4 (VBUS), P1.B9 (VBUS)
- net GND: now also J5.3 (Pin_3)
- net at U1.6 (RST/T2EX_/CAP2_): now also JP2.1 (A)
- new net: F1.1, P1.A4 (VBUS), P1.A9 (VBUS), P1.B4 (VBUS), P1.B9 (VBUS)
- no-connect marks 13 -> 12
Other:
- note added: "Testpoint"
- note removed: "HOST(CH552T)"
- moved on the sheet: R4, R5
