File: PCB/host.kicad_sch (KiCad schematic)
At the start: 13 parts, among them J5 Conn_01x03, P1 USB_C_Plug_USB2.0, U1 CH552T

Commit message: commit
Parts:
- added C4, C5, C6, C7, C8, C9: C, symbol Device:C
Connections:
- new net: C6.1, C7.1, C8.1, C9.1
- new net: C4.1, C5.1
