File: PCB/sleve.kicad_sch (KiCad schematic)
At the start: 4 parts, among them SW2 SW_Push, U2 CH32V003FxPx

Commit message: 基盤設計
Parts:
- added J6: Conn_01x05_Socket, Connector_PinHeader_2.54mm:PinHeader_1x05_P2.54mm_Vertical, symbol Connector:Conn_01x05_Socket
- added JP3: Jumper_2_Open, Jumper:SolderJumper-2_P1.3mm_Open_RoundedPad1.0x1.5mm, symbol Jumper:Jumper_2_Open
- added R6: 1k, Resistor_SMD:R_0603_1608Metric_Pad0.98x0.95mm_HandSolder, symbol Device:R
- D1: footprint LED_SMD:LED_Yuji_5730 -> LEDs:D_LED_5730
Connections:
- net +5V_{Slave}: now also J6.1 (Pin_1)
- net GND_{Slave}: now also J6.3 (Pin_3), JP3.2 (B), R6.2; no longer D1.1 (K)
- net LED: now reaches U2.16 (PC6)
- net LED: now also D1.2 (A)
- net SWDIO: now reaches U2.18 (PD1)
- net SWDIO: now also J6.4 (Pin_4)
- net TX: now reaches U2.2 (PD5)
- net TX: now also J6.2 (Pin_2)
- net RX: now reaches U2.3 (PD6)
- net RX: now also J6.5 (Pin_5)
- net at U2.4 (PD7): now also JP3.1 (A)
- net LED⇒ : no longer names the net of U2.5 (PA1)
- net LED⇒ : no longer D1.2 (A)
- new net: D1.1 (K), R6.1
- no-connect marks 12 -> 8
Other:
- note added: "DEBUG"
- note added: "POWER"
- moved on the sheet: C3, D1, SW2
